File: Co2-Sensor.sch (KiCad schematic (older format))
At the start: 70 parts, among them J1 OLED, J2 SCD30, J3 LED, J4 Power, J5 USB_C_Receptacle_USB2.0, J6 LED, J7 SPS30, J8 I2C, Q1 S8050, Q2 S8050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

Commit message: Add changes for Rev. 2
Parts:
- removed C1, C4: 100u/6.3V, Capacitor_Tantalum_SMD:CP_EIA-3528-15_AVX-H, symbol Device:CP_Small
- removed D7: Red, LED_SMD:LED_0603_1608Metric, symbol Device:LED_Small
- removed R21: 0R NC, Resistor_SMD:R_0603_1608Metric, symbol Device:R_Small
- removed R22: 0R, Resistor_SMD:R_0603_1608Metric, symbol Device:R_Small
- added C1, C4: 22u/25V, Capacitor_SMD:C_0805_2012Metric, symbol Device:C_Small
- added Q4: 2N7002, Package_TO_SOT_SMD:SOT-23, symbol Transistor_FET:BSS123
- added TP1, TP2: 5V, TestPoint:TestPoint_Pad_2.5x2.5mm, symbol Connector:TestPoint
- added TP3: LED1_CLK, TestPoint:TestPoint_Pad_2.5x2.5mm, symbol Connector:TestPoint
- added TP4: LED1_DATA, TestPoint:TestPoint_Pad_2.5x2.5mm, symbol Connector:TestPoint
- added TP5: LED2_CLK, TestPoint:TestPoint_Pad_2.5x2.5mm, symbol Connector:TestPoint
- added TP6: LED2_DATA, TestPoint:TestPoint_Pad_2.5x2.5mm, symbol Connector:TestPoint
- added TP7, TP8: GND, TestPoint:TestPoint_Pad_2.5x2.5mm, symbol Connector:TestPoint
- C7: value 1u/50V -> 2u2/16V; LCSC C15849 -> C23630
- F1: value 1A -> SMD1210-050; footprint Fuse:Fuse_0805_2012Metric -> Fuse:Fuse_1210_3225Metric; LCSC C70061 -> C70094
- R16: value 22R -> 4k7; LCSC C23345 -> C23162
- R18: value 47R -> 15k; LCSC C23182 -> C22809
- R19: value 330R -> 1k5; LCSC C23138 -> C22843
- R20: value 470R -> 12k; LCSC C23179 -> C22790
- R26, R6: value 470R -> 0R; LCSC C23179 -> C21189
Connections:
- net +3V3: now also R16.1, R20.1, C4.2; no longer R16.2
- net +5V: now also C3.2, C5.1, C8.1, R18.1; no longer C3.1, C5.2, C8.2, R18.2, R20.1
- net EN: now also C7.2, R26.1; no longer C7.1, R26.2
- net GND: now also C3.1, C5.2, C7.1, C8.2, R11.2, R14.2, C1.2, C4.1, Q4.2 (S), TP7.1, TP8.1; no longer C3.2, C5.1, C7.2, C8.1, D1.1 (K), D4.1 (K), R11.1, R14.1
- net IO2: now also R19.1; no longer R19.2
- net LED1_CLK: now also TP3.1
- net LED1_DATA: now also TP4.1
- net LED2_CLK: now also TP5.1
- net LED2_DATA: now also TP6.1
- net RXD: now also R5.1; no longer R5.2
- net SCL: now also U1.36 (IO22); no longer U1.7 (IO35)
- net SDA: now also U1.37 (IO23); no longer U1.6 (IO34)
- net SPS30_RX: now also R29.2; no longer R29.1
- net SPS30_TX: now also R31.2; no longer R31.1
- net TXD0: now also R5.2; no longer R5.1
- net VBUS: now also R13.1; no longer R13.2
- net ~DTR: now also R7.2; no longer R7.1
- net LED_DISABLE: now reaches U1.33 (IO21)
- net LED_DISABLE: now also R20.2, Q4.1 (G)
- net at C2.2, U3.6 (VDD): now also R15.2; no longer R15.1
- net at U3.9 (~RSTb): now also R15.1; no longer R15.2
- net at Q1.1 (B): now also R7.1; no longer R7.2
- net at D1.2 (A): now also R16.2; no longer R16.1
- net 5V_PREFUSE: now reaches J3.2 (Pin_2), J6.2 (Pin_2)
- net 5V_PREFUSE: now also D2.1 (K), D6.1 (K), F1.2, C1.1, TP1.1, TP2.1
- net at J5.B5 (CC2): now also R11.1; no longer R11.2
- net at D4.2 (A): now also R18.2; no longer R18.1
- net at D5.2 (A): now also R19.2; no longer R19.1
- net at Q3.3 (D): now also R26.2; no longer R26.1
- net at J7.2 (Pin_2), R30.1: now also R29.1; no longer R29.2
- net at J7.3 (Pin_3), R32.1: now also R31.1; no longer R31.2
- net IO0 renamed BUTTON4
- net IO12 renamed BUTTON1
- net BUTTON1: now also U1.6 (IO34); no longer U1.14 (IO12)
- net IO13 renamed BUTTON2
- net BUTTON2: now also U1.7 (IO35); no longer U1.16 (IO13)
- net IO15 renamed BUTTON3
- new net: R13.2, R14.1, U3.8 (VBUS)
- new net: D1.1 (K), D4.1 (K), Q4.3 (D)
- no-connect marks 31 -> 30
Other:
- moved on the sheet: D1, D4, D5, J3, J6, J8, R10, R16, R18, R19, R9

Commit message: Minor improvements
Parts:
- removed R2, R24, R28, R4: 470R, Resistor_SMD:R_0603_1608Metric, symbol Device:R_Small
- removed R26: 0R, Resistor_SMD:R_0603_1608Metric, symbol Device:R_Small
- added C10, C11, C12, C13: 100n/50V, Capacitor_SMD:C_0603_1608Metric, symbol Device:C_Small
- R1, R23, R25, R27, R3, R7, R8: value 12k -> 10k; LCSC C22790 -> C25804
Connections:
- net BUTTON1: now also SW1.1 (A), C10.2
- net BUTTON2: now also SW2.1 (A), C11.2
- net BUTTON3: now also SW3.1 (A), C12.2
- net BUTTON4: now also SW4.1 (A), C13.2
- net EN: now also Q3.3 (D)
- net GND: now also C10.1, C11.1, C12.1, C13.1
Changed lines of the file:
@@
 P 8100 4800
 F 0 "R7" V 7904 4800 50  0000 C CNN
-F 1 "12k" V 7995 4800 50  0000 C CNN
+F 1 "10k" V 7995 4800 50  0000 C CNN
 F 2 "Resistor_SMD:R_0603_1608Metric" H 8100 4800 50  0001 C CNN
 F 3 "~" H 8100 4800 50  0001 C CNN
-F 4 "C22790" V 8100 4800 50  0001 C CNN "LCSC"
+F 4 "C25804" V 8100 4800 50  0001 C CNN "LCSC"
 	1    8100 4800
 	0    -1   1    0
@@
 P 8100 5500
 F 0 "R8" V 7904 5500 50  0000 C CNN
-F 1 "12k" V 7995 5500 50  0000 C CNN
+F 1 "10k" V 7995 5500 50  0000 C CNN
 F 2 "Resistor_SMD:R_0603_1608Metric" H 8100 5500 50  0001 C CNN
 F 3 "~" H 8100 5500 50  0001 C CNN
-F 4 "C22790" V 8100 5500 50  0001 C CNN "LCSC"
+F 4 "C25804" V 8100 5500 50  0001 C CNN "LCSC"
 	1    8100 5500
 	0    1    1    0
@@
 P 3800 4700
 F 0 "R3" H 3741 4654 50  0000 R CNN
-F 1 "12k" H 3741 4745 50  0000 R CNN
+F 1 "10k" H 3741 4745 50  0000 R CNN
 F 2 "Resistor_SMD:R_0603_1608Metric" H 3800 4700 50  0001 C CNN
 F 3 "~" H 3800 4700 50  0001 C CNN
-F 4 "C22790" V 3800 4700 50  0001 C CNN "LCSC"
+F 4 "C25804" V 3800 4700 50  0001 C CNN "LCSC"
 	1    3800 4700
 	-1   0    0    1
@@
 P 3250 4700
 F 0 "R1" H 3191 4654 50  0000 R CNN
-F 1 "12k" H 3191 4745 50  0000 R CNN
+F 1 "10k" H 3191 4745 50  0000 R CNN
 F 2 "Resistor_SMD:R_0603_1608Metric" H 3250 4700 50  0001 C CNN
 F 3 "~" H 3250 4700 50  0001 C CNN
-F 4 "C22790" V 3250 4700 50  0001 C CNN "LCSC"
+F 4 "C25804" V 3250 4700 50  0001 C CNN "LCSC"
 	1    3250 4700
 	-1   0    0    1
 $EndComp
-$Comp
-L Device:R_Small R4
-U 1 1 5F5F99B8
-P 3800 5100
-F 0 "R4" H 3741 5054 50  0000 R CNN
-F 1 "470R" H 3741 5145 50  0000 R CNN
-F 2 "Resistor_SMD:R_0603_1608Metric" H 3800 5100 50  0001 C CNN
-F 3 "~" H 3800 5100 50  0001 C CNN
-F 4 "C23179" V 3800 5100 50  0001 C CNN "LCSC"
-	1    3800 5100
-	-1   0    0    1
-$EndComp
-$Comp
-L Device:R_Small R2
-U 1 1 5F5F9E8F
-P 3250 5100
-F 0 "R2" H 3191 5054 50  0000 R CNN
-F 1 "470R" H 3191 5145 50  0000 R CNN
-F 2 "Resistor_SMD:R_0603_1608Metric" H 3250 5100 50  0001 C CNN
-F 3 "~" H 3250 5100 50  0001 C CNN
-F 4 "C23179" V 3250 5100 50  0001 C CNN "LCSC"
-	1    3250 5100
-	-1   0    0    1
-$EndComp
-Wire Wire Line
-	3250 5200 3250 5300
-Wire Wire Line
-	3800 5300 3800 5200
 Wire Wire Line
 	3800 4800 3800 4900
@@
 	3250 4800 3250 4900
 Connection ~ 3250 4900
-Wire Wire Line
-	3250 4900 3250 5000
 Connection ~ 3800 4900
-Wire Wire Line
-	3800 4900 3800 5000
 $Comp
 L power:+3V3 #PWR0107
@@
 P 4350 4700
 F 0 "R23" H 4291 4654 50  0000 R CNN
-F 1 "12k" H 4291 4745 50  0000 R CNN
+F 1 "10k" H 4291 4745 50  0000 R CNN
 F 2 "Resistor_SMD:R_0603_1608Metric" H 4350 4700 50  0001 C CNN
 F 3 "~" H 4350 4700 50  0001 C CNN
-F 4 "C22790" V 4350 4700 50  0001 C CNN "LCSC"
+F 4 "C25804" V 4350 4700 50  0001 C CNN "LCSC"
 	1    4350 4700
 	-1   0    0    1
 $EndComp
-$Comp
-L Device:R_Small R24
-U 1 1 5FB032FA
-P 4350 5100
-F 0 "R24" H 4291 5054 50  0000 R CNN
-F 1 "470R" H 4291 5145 50  0000 R CNN
-F 2 "Resistor_SMD:R_0603_1608Metric" H 4350 5100 50  0001 C CNN
-F 3 "~" H 4350 5100 50  0001 C CNN
-F 4 "C23179" V 4350 5100 50  0001 C CNN "LCSC"
-	1    4350 5100
-	-1   0    0    1
-$EndComp
-Wire Wire Line
-	4350 5300 4350 5200
 Wire Wire Line
 	4350 4800 4350 4900
 Connection ~ 4350 4900
-Wire Wire Line
-	4350 4900 4350 5000
 $Comp
 L power:+3V3 #PWR0154
@@
 P 4900 4700
 F 0 "R27" H 4841 4654 50  0000 R CNN
-F 1 "12k" H 4841 4745 50  0000 R CNN
+F 1 "10k" H 4841 4745 50  0000 R CNN
 F 2 "Resistor_SMD:R_0603_1608Metric" H 4900 4700 50  0001 C CNN
 F 3 "~" H 4900 4700 50  0001 C CNN
-F 4 "C22790" V 4900 4700 50  0001 C CNN "LCSC"
+F 4 "C25804" V 4900 4700 50  0001 C CNN "LCSC"
 	1    4900 4700
 	-1   0    0    1
 $EndComp
-$Comp
-L Device:R_Small R28
-U 1 1 5FBD4C55
-P 4900 5100
-F 0 "R28" H 4841 5054 50  0000 R CNN
-F 1 "470R" H 4841 5145 50  0000 R CNN
-F 2 "Resistor_SMD:R_0603_1608Metric" H 4900 5100 50  0001 C CNN
-F 3 "~" H 4900 5100 50  0001 C CNN
-F 4 "C23179" V 4900 5100 50  0001 C CNN "LCSC"
-	1    4900 5100
-	-1   0    0    1
-$EndComp
-Wire Wire Line
-	4900 5300 4900 5200
 Wire Wire Line
 	4900 4800 4900 4900
 Connection ~ 4900 4900
-Wire Wire Line
-	4900 4900 4900 5000
 $Comp
 L power:+3V3 #PWR0156
@@
 $EndComp
 $Comp
-L Device:R_Small R26
-U 1 1 5FC1BD90
-P 2200 3800
-F 0 "R26" H 2141 3754 50  0000 R CNN
-F 1 "0R" H 2141 3845 50  0000 R CNN
-F 2 "Resistor_SMD:R_0603_1608Metric" H 2200 3800 50  0001 C CNN
-F 3 "~" H 2200 3800 50  0001 C CNN
-F 4 "C21189" V 2200 3800 50  0001 C CNN "LCSC"
-	1    2200 3800
-	-1   0    0    -1
-$EndComp
-$Comp
 L Device:R_Small R25
 U 1 1 5FC2CBCC
 P 2200 3400
 F 0 "R25" H 2141 3354 50  0000 R CNN
-F 1 "12k" H 2141 3445 50  0000 R CNN
+F 1 "10k" H 2141 3445 50  0000 R CNN
 F 2 "Resistor_SMD:R_0603_1608Metric" H 2200 3400 50  0001 C CNN
 F 3 "~" H 2200 3400 50  0001 C CNN
-F 4 "C22790" V 2200 3400 50  0001 C CNN "LCSC"
+F 4 "C25804" V 2200 3400 50  0001 C CNN "LCSC"
 	1    2200 3400
 	-1   0    0    1
@@
 Text Label 2050 3600 0    50   ~ 0
 EN
-Wire Wire Line
-	2200 4000 2200 3900
-Wire Wire Line
-	2200 3700 2200 3600
 Wire Wire Line
 	2200 3600 2050 3600
@@
 BUTTON1
 Wire Wire Line
-	2900 4900 3250 4900
+	2900 4900 3000 4900
 Text Label 3450 4900 0    50   ~ 0
 BUTTON2
 Wire Wire Line
-	3450 4900 3800 4900
+	3450 4900 3550 4900
 Text Label 750  4150 0    50   ~ 0
 BUTTON1
@@
 BUTTON3
 Wire Wire Line
-	4000 4900 4350 4900
+	4000 4900 4100 4900
 Text Label 8500 2050 2    50   ~ 0
 BUTTON3
@@
 BUTTON4
 Wire Wire Line
-	4550 4900 4900 4900
+	4550 4900 4650 4900
 Text Label 7600 6050 1    50   ~ 0
 BUTTON4
@@
 	1    0    0    -1
 $EndComp
+Wire Wire Line
+	3250 4900 3250 5300
+Wire Wire Line
+	3800 4900 3800 5300
+Wire Wire Line
+	4350 4900 4350 5300
+Wire Wire Line
+	4900 4900 4900 5300
+$Comp
+L Device:C_Small C10
+U 1 1 5F7E27EA
+P 3000 5100
+F 0 "C10" H 2909 5054 50  0000 R CNN
+F 1 "100n/50V" H 2909 5145 50  0000 R CNN
+F 2 "Capacitor_SMD:C_0603_1608Metric" H 3000 5100 50  0001 C CNN
+F 3 "~" H 3000 5100 50  0001 C CNN
+F 4 "C24452" H 3000 5100 50  0001 C CNN "LCSC"
+	1    3000 5100
+	-1   0    0    1
+$EndComp
+$Comp
+L power:GND #PWR0120
+U 1 1 5F7E37C3
+P 3000 5800
+F 0 "#PWR0120" H 3000 5550 50  0001 C CNN
+F 1 "GND" H 3005 5627 50  0000 C CNN
+F 2 "" H 3000 5800 50  0001 C CNN
+F 3 "" H 3000 5800 50  0001 C CNN
+	1    3000 5800
+	1    0    0    -1
+$EndComp
+Wire Wire Line
+	3000 5800 3000 5200
+Wire Wire Line
+	3000 5000 3000 4900
+Connection ~ 3000 4900
+Wire Wire Line
+	3000 4900 3250 4900
+$Comp
+L Device:C_Small C11
+U 1 1 5F816C68
+P 3550 5100
+F 0 "C11" H 3459 5054 50  0000 R CNN
+F 1 "100n/50V" H 3459 5145 50  0000 R CNN
+F 2 "Capacitor_SMD:C_0603_1608Metric" H 3550 5100 50  0001 C CNN
+F 3 "~" H 3550 5100 50  0001 C CNN
+F 4 "C24452" H 3550 5100 50  0001 C CNN "LCSC"
+	1    3550 5100
+	-1   0    0    1
+$EndComp
+Wire Wire Line
+	3550 4900 3550 5000
+Connection ~ 3550 4900
+Wire Wire Line
+	3550 4900 3800 4900
+$Comp
+L Device:C_Small C12
+U 1 1 5F828DF4
+P 4100 5100
+F 0 "C12" H 4009 5054 50  0000 R CNN
+F 1 "100n/50V" H 4009 5145 50  0000 R CNN
+F 2 "Capacitor_SMD:C_0603_1608Metric" H 4100 5100 50  0001 C CNN
+F 3 "~" H 4100 5100 50  0001 C CNN
+F 4 "C24452" H 4100 5100 50  0001 C CNN "LCSC"
+	1    4100 5100
+	-1   0    0    1
+$EndComp
+Wire Wire Line
+	4100 5000 4100 4900
+Connection ~ 4100 4900
+Wire Wire Line
+	4100 4900 4350 4900
+$Comp
+L Device:C_Small C13
+U 1 1 5F83B2FD
+P 4650 5100
+F 0 "C13" H 4559 5054 50  0000 R CNN
+F 1 "100n/50V" H 4559 5145 50  0000 R CNN
+F 2 "Capacitor_SMD:C_0603_1608Metric" H 4650 5100 50  0001 C CNN
+F 3 "~" H 4650 5100 50  0001 C CNN
+F 4 "C24452" H 4650 5100 50  0001 C CNN "LCSC"
+	1    4650 5100
+	-1   0    0    1
+$EndComp
+Wire Wire Line
+	4650 5000 4650 4900
+Connection ~ 4650 4900
+Wire Wire Line
+	4650 4900 4900 4900
+Wire Wire Line
+	3550 5200 3550 5800
+Wire Wire Line
+	4100 5200 4100 5800
+Wire Wire Line
+	4650 5200 4650 5800
+$Comp
+L power:GND #PWR0142
+U 1 1 5F886353
+P 3550 5800
+F 0 "#PWR0142" H 3550 5550 50  0001 C CNN
+F 1 "GND" H 3555 5627 50  0000 C CNN
+F 2 "" H 3550 5800 50  0001 C CNN
+F 3 "" H 3550 5800 50  0001 C CNN
+	1    3550 5800
+	1    0    0    -1
+$EndComp
+$Comp
+L power:GND #PWR0151
+U 1 1 5F88671C
+P 4100 5800
+F 0 "#PWR0151" H 4100 5550 50  0001 C CNN
+F 1 "GND" H 4105 5627 50  0000 C CNN
+F 2 "" H 4100 5800 50  0001 C CNN
+F 3 "" H 4100 5800 50  0001 C CNN
+	1    4100 5800
+	1    0    0    -1
+$EndComp
+$Comp
+L power:GND #PWR0152
+U 1 1 5F886A5D
+P 4650 5800
+F 0 "#PWR0152" H 4650 5550 50  0001 C CNN
+F 1 "GND" H 4655 5627 50  0000 C CNN
+F 2 "" H 4650 5800 50  0001 C CNN
+F 3 "" H 4650 5800 50  0001 C CNN
+	1    4650 5800
+	1    0    0    -1
+$EndComp
+Wire Wire Line
+	2200 3600 2200 4000
 $EndSCHEMATC
